File: PCB/palmpadpcb.kicad_pcb (KiCad board)
At the start: 2 copper layers, 100 x 100 mm, 140 parts, among them J1 5V_Control, J10 ENC2_A, J11 ENC2_B, J12 ENC_OUT, J13 ENC_OUT, J14 Row1, J15 Row1, J16 Row2, J17 Row3, J18 Row3, J19 Row2, J2 5V_Control, J20 Row3_Jump, J21 Row3_Jump, J22 Col1_Jump1, J23 Col1_Jump1, J24 Col1_Jump2, J25 Col1_Jump2, J26 Col1_OUT, J27 Col1_OUT, J28 Col2_OUT, J29 Col2_OUT, J3 GND_Control, J30 Col2_Jump1, J31 Col2_Jump1, J32 Col2_Jump2, J33 Col2_Jump2, J34 Col3_Jump2, J35 Col3_Jump2, J36 Col3_Jump1, J37 Col3_Jump1, J38 Col3_OUT, J39 Col3_OUT, J4 GND_Control, J40 Col4_OUT, J41 Col4_OUT, J42 Col4_Jump1, J43 Col4_Jump1, J44 Col4_Jump2, J45 Col4_Jump2, J46 SCL, J47 SDA, J48 SDA, J5 SCL, J6 GND_ENC1, J7 GND_ENC2, J8 ENC1_B, J9 ENC1_A, SW1 SW_Push, SW10 SW_Push, SW11 SW_Push, SW12 SW_Push, SW15 SW_Push, SW16 SW_Push, SW2 SW_Push, SW3 SW_Push, SW4 SW_Push, SW5 SW_Push, SW6 SW_Push, SW7 SW_Push, SW8 SW_Push, SW9 SW_Push, U1 MOUDLE-SEEEDUINO-XIAO, U2 ER_OLEDM0.91_1x-I2C

Commit message: Revision 2
Parts:
- D13, D14, D15, D16, D17, D18, D19, D20, D21, D22, D23, D24, D25, D26, D27, D28, J13, J14, J16, J17, J2, J26, J28, J39, J4, J40, J47, J5, U1: moved to B.Cu
- moved D13 16.5 mm to (145.8, 91.7)
- moved D14 16.5 mm to (145.8, 102.2)
- moved D15 16.5 mm to (145.8, 113.0)
- moved D16 16.5 mm to (145.8, 123.0)
- moved D17 16.5 mm to (145.8, 132.7)
- moved D26 16.5 mm to (162.2, 112.8)
- moved D27 16.5 mm to (162.2, 102.7)
- moved D24 16.0 mm to (162.0, 132.8)
- moved D25 16.0 mm to (162.0, 123.0)
- moved D28 16.0 mm to (162.0, 92.0)
- moved D18 7.00 mm to (150.5, 132.7)
- moved D19 7.00 mm to (150.5, 123.0)
- moved D20 7.00 mm to (150.5, 113.0)
- moved J14 7.00 mm to (150.5, 100.5), turned to 0 degrees
- moved J16 7.00 mm to (150.5, 97.0), turned to 0 degrees
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Routing:
- net Col2: track 163.2 -> 187.3 mm, vias 0 -> 1
- net GND: track 366.1 -> 388.5 mm, vias 4 -> 5
- net Col1: track 190.3 -> 211.9 mm, vias 0 -> 1
- net Row1: track 121.7 -> 107.0 mm
- net Col3: track 160.9 -> 173.2 mm, vias 0 -> 1
- net Row2: track 137.2 -> 125.3 mm, vias 0 -> 1
- net Col4: track 128.2 -> 120.3 mm, vias 0 -> 1
- net Row3: track 163.7 -> 157.6 mm, vias 0 -> 1
- net 5V: track 372.1 -> 366.9 mm, vias 2 -> 1
- net SCL: track 115.4 -> 117.7 mm, vias 0 -> 1
- net SDA: track 116.6 -> 118.7 mm, vias 1 -> 0
- net ENC: track 140.6 -> 142.0 mm, vias 2 -> 1
Other:
- outline, holes or cut-outs redrawn
